Commit message: Use collada file for pokeball display.

File: urdf/ur_benchmark/pokeball.urdf (robot description, URDF)
Before this commit: robot pokeball, 1 links, 0 joints
Links:
- link base_link: geometry collision sphere radius=0.025; visual mesh filename=package://hpp_environments/meshes/ur_benchmark/pokeball.dae scale=0.025 0.025 0.025

Commit message: Use box for collision geometry of pokeball

File: urdf/ur_benchmark/pokeball.urdf (robot description, URDF)
Before this commit: robot pokeball, 1 links, 0 joints
Links:
- link base_link: geometry collision box size=0.025 0.025 0.025; visual mesh filename=package://hpp_environments/meshes/ur_benchmark/pokeball.dae scale=0.025 0.025 0.025
