Commit message: Add texture file for Romeo logo and set placard to color of logo.
  - texture does not display well in gepetto-gui.

File: urdf/placard-vertical.urdf (robot description, URDF)
Before this commit: robot placard, 5 links, 4 joints
Links:
- link placard: geometry collision cylinder length=1.4 radius=0.015; visual box size=0.01 0.62 0.3

File: urdf/placard.urdf (robot description, URDF)
Before this commit: robot placard, 1 links, 0 joints
Links:
- link placard: geometry collision cylinder length=1.4 radius=0.015; visual box size=0.01 0.62 0.3
