Commit message: [buggy.urdf] Add collision geometry for front wheels.

File: urdf/buggy.urdf (robot description, URDF)
Before this commit: robot buggy, 3 links, 2 joints
Links:
- link wheel_frontleft: geometry collision mesh filename=package://hpp_environments/meshes/buggy/wheel_frontleft.dae; visual mesh filename=package://hpp_environments/meshes/buggy/wheel_frontleft.dae
- link wheel_frontright: geometry collision mesh filename=package://hpp_environments/meshes/buggy/wheel_frontright.dae; visual mesh filename=package://hpp_environments/meshes/buggy/wheel_frontright.dae
