Commit message: Add cylinders with two different lengths.

File: urdf/construction_set/cylinder_13.urdf (robot description, URDF)
Before this commit: robot cylinder, 1 links, 0 joints
Links:
- link base_link: geometry collision box size=0.12970562748477143 0.01 0.01; visual cylinder length=0.12970562748477143 radius=0.01
