Commit message: desk model complete

File: urdf/drawer_desk/desk.urdf (robot description, URDF)
Before this commit: robot desk, 10 links, 9 joints
Links:
- added link upper_drawer_background; collision box size=0.783333333333 0.025 0.175; visual box size=0.783333333333 0.025 0.175
- added link upper_drawer_bottom; collision box size=0.783333333333 0.75 0.025; visual box size=0.783333333333 0.75 0.025
- added link upper_drawer_front; collision box size=0.833333333333 0.025 0.225; visual box size=0.833333333333 0.025 0.225
- added link upper_drawer_handle; collision sphere radius=0.025; visual sphere radius=0.025
- added link upper_drawer_left; collision box size=0.025 0.725 0.175; visual box size=0.025 0.725 0.175
- added link upper_drawer_right; collision box size=0.025 0.725 0.175; visual box size=0.025 0.725 0.175
Joints:
- added joint upper_case_bottom_upper_drawer_bottom_joint: type prismatic, parent upper_case_bottom, child upper_drawer_bottom, origin xyz=0 -0.0125 0.025 rpy=0 0 0, axis 0 1 0, limit lower=-0.3875 upper=0 effort=500 velocity=0.5
- added joint upper_drawer_bottom_background_joint: type fixed, parent upper_drawer_bottom, child upper_drawer_background, origin xyz=0 0.3625 0.1 rpy=0 0 0
- added joint upper_drawer_bottom_front_joint: type fixed, parent upper_drawer_bottom, child upper_drawer_front, origin xyz=0 -0.3875 0.075 rpy=0 0 0
- added joint upper_drawer_bottom_left_joint: type fixed, parent upper_drawer_bottom, child upper_drawer_left, origin xyz=-0.379166666666 -0.0125 0.1 rpy=0 0 0
- added joint upper_drawer_bottom_right_joint: type fixed, parent upper_drawer_bottom, child upper_drawer_right, origin xyz=0.379166666666 -0.0125 0.1 rpy=0 0 0
- added joint upper_drawer_front_handle_joint: type fixed, parent upper_drawer_front, child upper_drawer_handle, origin xyz=0 -0.0375 0 rpy=0 0 0

File: urdf/drawer_desk/desk.urdf.xacro (robot description, xacro)
@@ -3,4 +3,5 @@
 	<xacro:include filename="table.urdf.xacro"/>
 	<xacro:include filename="case.urdf.xacro"/>
+	<xacro:include filename="drawer.urdf.xacro"/>
 	<link name="world"/>
 	<xacro:property name="board_h" value="0.6"/>
@@ -22,3 +23,11 @@
 		<origin xyz="${(board_sX/2) - ((board_sX/3)/2) - (leg_foot_sX)} ${planks_width/2} ${(-board_sZ/2) - ((board_h/3)/2)}" rpy="0 0 0"/>
 	</joint>
+	<xacro:drawer prefix="upper" planks_thickness="${planks_width}" drawer_sizeX="${board_sX/3}" drawer_sizeY="${(board_sY/2) + planks_width}" drawer_sizeZ="${(board_h/3) + planks_width}" drawer_handle_radius="0.025"/>
+	<joint name="upper_case_bottom_upper_drawer_bottom_joint" type="prismatic">
+		<parent link="upper_case_bottom"/>
+		<child link="upper_drawer_bottom"/>
+		<limit effort="500" lower="${-(((board_sY/2) + planks_width)/2)}" upper="0" velocity="0.5"/>
+		<axis xyz="0 1 0"/>
+		<origin xyz="0 ${-planks_width/2} ${planks_width}" rpy="0 0 0"/>
+	</joint>
 </robot>

File: urdf/drawer_desk/drawer.urdf.xacro (robot description, xacro)
@@ -11,5 +11,5 @@
 			<visual>
 				<geometry>
-					<box size="${} ${} ${}"/>
+					<box size="${drawer_sizeX - (2*planks_thickness)} ${drawer_sizeY - planks_thickness} ${planks_thickness}"/>
 				</geometry>
 				<origin xyz="0 0 0" rpy="0 0 0"/>
@@ -18,5 +18,5 @@
 			<collision>
 				<geometry>
-					<box size="${} ${} ${}"/>
+					<box size="${drawer_sizeX - (2*planks_thickness)} ${drawer_sizeY - planks_thickness} ${planks_thickness}"/>
 				</geometry>
 				<origin xyz="0 0 0" rpy="0 0 0"/>
@@ -26,5 +26,5 @@
 			<visual>
 				<geometry>
-					<box size="${} ${} ${}"/>
+					<box size="${drawer_sizeX - (2*planks_thickness)} ${planks_thickness} ${drawer_sizeZ - (2*planks_thickness)}"/>
 				</geometry>
 				<origin xyz="0 0 0" rpy="0 0 0"/>
@@ -33,5 +33,5 @@
 			<collision>
 				<geometry>
-					<box size="${} ${} ${}"/>
+					<box size="${drawer_sizeX - (2*planks_thickness)} ${planks_thickness} ${drawer_sizeZ - (2*planks_thickness)}"/>
 				</geometry>
 				<origin xyz="0 0 0" rpy="0 0 0"/>
@@ -41,10 +41,10 @@
 			<parent link="${prefix}_drawer_bottom"/>
 			<child link="${prefix}_drawer_background"/>
-			<origin xyz="" rpy="0 0 0"/>
+			<origin xyz="0 ${((drawer_sizeY - planks_thickness)/2) - (planks_thickness/2)} ${((drawer_sizeZ - (2*planks_thickness))/2) + (planks_thickness/2)}" rpy="0 0 0"/>
 		</joint>
 		<link name="${prefix}_drawer_right">
 			<visual>
 				<geometry>
-					<box size="${} ${} ${}"/>
+					<box size="${planks_thickness} ${drawer_sizeY - (2*planks_thickness)} ${drawer_sizeZ - (2*planks_thickness)}"/>
 				</geometry>
 				<origin xyz="0 0 0" rpy="0 0 0"/>
@@ -53,5 +53,5 @@
 			<collision>
 				<geometry>
-					<box size="${} ${} ${}"/>
+					<box size="${planks_thickness} ${drawer_sizeY - (2*planks_thickness)} ${drawer_sizeZ - (2*planks_thickness)}"/>
 				</geometry>
 				<origin xyz="0 0 0" rpy="0 0 0"/>
@@ -61,10 +61,10 @@
 			<parent link="${prefix}_drawer_bottom"/>
 			<child link="${prefix}_drawer_right"/>
-			<origin xyz="" rpy="0 0 0"/>
+			<origin xyz="${((drawer_sizeX - (2*planks_thickness))/2) - (planks_thickness/2)} ${-planks_thickness/2} ${((drawer_sizeZ - (2*planks_thickness))/2) + (planks_thickness/2)}" rpy="0 0 0"/>
 		</joint>
 		<link name="${prefix}_drawer_left">
 			<visual>
 				<geometry>
-					<box size="${} ${} ${}"/>
+					<box size="${planks_thickness} ${drawer_sizeY - (2*planks_thickness)} ${drawer_sizeZ - (2*planks_thickness)}"/>
 				</geometry>
 				<origin xyz="0 0 0" rpy="0 0 0"/>
@@ -73,5 +73,5 @@
 			<collision>
 				<geometry>
-					<box size="${} ${} ${}"/>
+					<box size="${planks_thickness} ${drawer_sizeY - (2*planks_thickness)} ${drawer_sizeZ - (2*planks_thickness)}"/>
 				</geometry>
 				<origin xyz="0 0 0" rpy="0 0 0"/>
@@ -81,10 +81,10 @@
 			<parent link="${prefix}_drawer_bottom"/>
 			<child link="${prefix}_drawer_left"/>
-			<origin xyz="" rpy="0 0 0"/>
+			<origin xyz="${-((drawer_sizeX - (2*planks_thickness))/2) + (planks_thickness/2)} ${-planks_thickness/2} ${((drawer_sizeZ - (2*planks_thickness))/2) + (planks_thickness/2)}" rpy="0 0 0"/>
 		</joint>
 		<link name="${prefix}_drawer_front">
 			<visual>
 				<geometry>
-					<box size="${} ${} ${}"/>
+					<box size="${drawer_sizeX} ${planks_thickness} ${drawer_sizeZ}"/>
 				</geometry>
 				<origin xyz="0 0 0" rpy="0 0 0"/>
@@ -93,5 +93,5 @@
 			<collision>
 				<geometry>
-					<box size="${} ${} ${}"/>
+					<box size="${drawer_sizeX} ${planks_thickness} ${drawer_sizeZ}"/>
 				</geometry>
 				<origin xyz="0 0 0" rpy="0 0 0"/>
@@ -101,5 +101,5 @@
 			<parent link="${prefix}_drawer_bottom"/>
 			<child link="${prefix}_drawer_front"/>
-			<origin xyz="" rpy="0 0 0"/>
+			<origin xyz="0 ${-((drawer_sizeY - planks_thickness)/2) - (planks_thickness/2)} ${(drawer_sizeZ/2) - (3*planks_thickness/2)}" rpy="0 0 0"/>
 		</joint>
 		<link name="${prefix}_drawer_handle">
@@ -121,5 +121,5 @@
 			<parent link="${prefix}_drawer_front"/>
 			<child link="${prefix}_drawer_handle"/>
-			<origin xyz="" rpy="0 0 0"/>
+			<origin xyz="0 ${-drawer_handle_radius - (planks_thickness/2)} 0" rpy="0 0 0"/>
 		</joint>
 	</xacro:macro>

Commit message: Desk model: ground added

File: urdf/drawer_desk/desk.urdf (robot description, URDF)
Before this commit: robot desk, 16 links, 15 joints
Links:
- added link ground; collision box size=5 5 0.1; visual box size=5 5 0.1
Joints:
- added joint world_ground_joint: type fixed, parent world, child ground, origin xyz=0 0 -0.05 rpy=0 0 0

File: urdf/drawer_desk/desk.urdf.xacro (robot description, xacro)
@@ -4,5 +4,29 @@
 	<xacro:include filename="case.urdf.xacro"/>
 	<xacro:include filename="drawer.urdf.xacro"/>
+	<xacro:property name="ground_thickness" value="0.1"/>
+	<material name="black">
+		<color rgba="0.05 0.05 0.05 1"/>
+	</material>
 	<link name="world"/>
+	<link name="ground">
+		<visual>
+			<geometry>
+				<box size="5 5 ${ground_thickness}"/>
+			</geometry>
+			<origin xyz="0 0 0" rpy="0 0 0"/>
+			<material name="black"/>
+		</visual>
+		<collision>
+			<geometry>
+				<box size="5 5 ${ground_thickness}"/>
+			</geometry>
+			<origin xyz="0 0 0" rpy="0 0 0"/>
+		</collision>
+	</link>
+	<joint name="world_ground_joint" type="fixed">
+		<parent link="world"/>
+		<child link="ground"/>
+		<origin xyz="0 0 ${-ground_thickness/2}" rpy="0 0 0"/>
+	</joint>
 	<xacro:property name="board_h" value="0.6"/>
 	<xacro:property name="board_sX" value="2.5"/>

Commit message: table elevation

File: urdf/drawer_desk/desk.urdf (robot description, URDF)
Before this commit: robot desk, 17 links, 16 joints
Links:
- link left_body: geometry collision cylinder length=0.65 radius=0.025; visual cylinder length=0.65 radius=0.025
- link right_body: geometry collision cylinder length=0.65 radius=0.025; visual cylinder length=0.65 radius=0.025
- link upper_case_background: geometry collision box size=0.833333333333 0.025 0.233333333333; visual box size=0.833333333333 0.025 0.233333333333
- link upper_case_left: geometry collision box size=0.025 0.75 0.233333333333; visual box size=0.025 0.75 0.233333333333
- link upper_case_right: geometry collision box size=0.025 0.75 0.233333333333; visual box size=0.025 0.75 0.233333333333
- link upper_drawer_background: geometry collision box size=0.783333333333 0.025 0.208333333333; visual box size=0.783333333333 0.025 0.208333333333
- link upper_drawer_front: geometry collision box size=0.833333333333 0.025 0.258333333333; visual box size=0.833333333333 0.025 0.258333333333
- link upper_drawer_left: geometry collision box size=0.025 0.725 0.208333333333; visual box size=0.025 0.725 0.208333333333
- link upper_drawer_right: geometry collision box size=0.025 0.725 0.208333333333; visual box size=0.025 0.725 0.208333333333
Joints:
- joint board_left_body_joint: origin xyz=-1.225 0 -0.3 rpy=0 0 0 -> xyz=-1.225 0 -0.35 rpy=0 0 0
- joint board_right_body_joint: origin xyz=1.225 0 -0.3 rpy=0 0 0 -> xyz=1.225 0 -0.35 rpy=0 0 0
- joint board_upper_case_background_joint: origin xyz=0.783333333333 0.0125 -0.125 rpy=0 0 0 -> xyz=0.783333333333 0.0125 -0.141666666667 rpy=0 0 0
- joint left_body_foot_joint: origin xyz=0 0 -0.2875 rpy=0 0 0 -> xyz=0 0 -0.3375 rpy=0 0 0
- joint right_body_foot_joint: origin xyz=0 0 -0.2875 rpy=0 0 0 -> xyz=0 0 -0.3375 rpy=0 0 0
- joint upper_case_background_bottom_joint: origin xyz=0 -0.375 -0.1125 rpy=0 0 0 -> xyz=0 -0.375 -0.129166666667 rpy=0 0 0
- joint upper_drawer_bottom_background_joint: origin xyz=0 0.3625 0.1 rpy=0 0 0 -> xyz=0 0.3625 0.116666666667 rpy=0 0 0
- joint upper_drawer_bottom_front_joint: origin xyz=0 -0.3875 0.075 rpy=0 0 0 -> xyz=0 -0.3875 0.0916666666665 rpy=0 0 0
- joint upper_drawer_bottom_left_joint: origin xyz=-0.379166666666 -0.0125 0.1 rpy=0 0 0 -> xyz=-0.379166666666 -0.0125 0.116666666667 rpy=0 0 0
- joint upper_drawer_bottom_right_joint: origin xyz=0.379166666666 -0.0125 0.1 rpy=0 0 0 -> xyz=0.379166666666 -0.0125 0.116666666667 rpy=0 0 0
- joint world_board_joint: origin xyz=0 0 0.6 rpy=0 0 0 -> xyz=0 0 0.7 rpy=0 0 0

File: urdf/drawer_desk/desk.urdf.xacro (robot description, xacro)
@@ -29,5 +29,5 @@
 		<origin xyz="0 0 ${-ground_thickness/2}" rpy="0 0 0"/>
 	</joint>
-	<xacro:property name="board_h" value="0.6"/>
+	<xacro:property name="board_h" value="0.7"/>
 	<xacro:property name="board_sX" value="2.5"/>
 	<xacro:property name="board_sY" value="1.5"/>
