Commit message: change all paths in urdf from rbprm to hpp_environments

File: urdf/multicontact/bauzil_stairs.urdf (robot description, URDF)
Before this commit: robot stair_bauzil, 1 links, 0 joints
Links:
- link base_link: geometry collision mesh filename=package://hpp_environments/meshes/multicontact/bauzil_stair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; visual mesh filename=package://hpp_environments/meshes/multicontact/bauzil_stair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

File: urdf/multicontact/bauzil_stairs_10cm.urdf (robot description, URDF)
Before this commit: robot stair_bauzil, 1 links, 0 joints
Links:
- link base_link: geometry collision mesh filename=package://hpp_environments/meshes/multicontact/bauzil_stair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; visual mesh filename=package://hpp_environments/meshes/multicontact/bauzil_stair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

File: urdf/multicontact/bauzil_stairs_collision.urdf (robot description, URDF)
Before this commit: robot stair_bauzil, 1 links, 0 joints
Links:
- link base_link: geometry collision mesh filename=package://hpp_environments/meshes/multicontact/bauzil_stair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; visual mesh filename=package://hpp_environments/meshes/multicontact/bauzil_stair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

File: urdf/multicontact/box.urdf (robot description, URDF)
Before this commit: robot box, 1 links, 0 joints
Links:
- link base_link: geometry collision mesh filename=package://hpp_environments/meshes/multicontact/box.stl; visual mesh filename=package://hpp_environments/meshes/multicontact/robot_box.stl

File: urdf/multicontact/box_rom.urdf (robot description, URDF)
Before this commit: robot box, 1 links, 0 joints
Links:
- link base_link: geometry collision mesh filename=package://hpp_environments/meshes/multicontact/box_rom.stl; visual mesh filename=package://hpp_environments/meshes/multicontact/box_rom.stl

File: urdf/multicontact/bridge_towr.urdf (robot description, URDF)
Before this commit: robot stair_bauzil, 1 links, 0 joints
Links:
- link base_link: geometry collision mesh filename=package://hpp_environments/meshes/multicontact/bridge.stl; visual mesh filename=package://hpp_environments/meshes/multicontact/bridge.stl

File: urdf/multicontact/car.urdf (robot description, URDF)
Before this commit: robot car, 1 links, 0 joints
Links:
- link base_link: geometry collision mesh filename=package://hpp_environments/meshes/multicontact/car.stl; visual mesh filename=package://hpp_environments/meshes/multicontact/car.stl

File: urdf/multicontact/climb.urdf (robot description, URDF)
Before this commit: robot climb, 1 links, 0 joints
Links:
- link base_link: geometry collision mesh filename=package://hpp_environments/meshes/multicontact/climb.stl; visual mesh filename=package:///../hpp-rbprm-corba/meshes/climb.stl

File: urdf/multicontact/cross_gap.urdf (robot description, URDF)
Before this commit: robot cross_gap, 1 links, 0 joints
Links:
- link base_link: geometry collision mesh filename=package://hpp_environments/meshes/multicontact/cross_gap2.s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; visual mesh filename=package://hpp_environments/meshes/multicontact/cross_gap2.s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

File: urdf/multicontact/cubeWorld3.urdf (robot description, URDF)
Before this commit: robot cubeWorld, 1 links, 0 joints
Links:
- link base_link: geometry collision mesh filename=package://hpp_environments/meshes/multicontact/cubeWorld3.s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; visual mesh filename=package://hpp_environments/meshes/multicontact/cubeWorld3.s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

File: urdf/multicontact/cubeWorld_nonCoplanar.urdf (robot description, URDF)
Before this commit: robot cubeWorld, 1 links, 0 joints
Links:
- link base_link: geometry collision mesh filename=package://hpp_environments/meshes/multicontact/cube_non_cop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; visual mesh filename=package://hpp_environments/meshes/multicontact/cube_non_cop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

File: urdf/multicontact/cubeWorld_nonCoplanar2.urdf (robot description, URDF)
Before this commit: robot cubeWorld, 1 links, 0 joints
Links:
- link base_link: geometry collision mesh filename=package://hpp_environments/meshes/multicontact/cube_non_cop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; visual mesh filename=package://hpp_environments/meshes/multicontact/cube_non_cop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

File: urdf/multicontact/darpa.urdf (robot description, URDF)
Before this commit: robot chair, 1 links, 0 joints
Links:
- link base_link: geometry collision mesh filename=package://hpp_environments/meshes/multicontact/darpareduced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; visual mesh filename=package://hpp_environments/meshes/multicontact/darpareduced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

File: urdf/multicontact/darpa_no_ctc_mid.urdf (robot description, URDF)
Before this commit: robot chair, 1 links, 0 joints
Links:
- link base_link: geometry collision mesh filename=package://hpp_environments/meshes/multicontact/darpa_no_ctc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; visual mesh filename=package://hpp_environments/meshes/multicontact/darpa_no_ctc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

File: urdf/multicontact/darpa_no_mid.urdf (robot description, URDF)
Before this commit: robot chair, 1 links, 0 joints
Links:
- link base_link: geometry collision mesh filename=package://hpp_environments/meshes/multicontact/darpa_no_mid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; visual mesh filename=package://hpp_environments/meshes/multicontact/darpa_no_mid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

File: urdf/multicontact/downSlope.urdf (robot description, URDF)
Before this commit: robot stair_bauzil, 1 links, 0 joints
Links:
- link base_link: geometry collision mesh filename=package://hpp_environments/meshes/multicontact/downSlope2.s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; visual mesh filename=package://hpp_environments/meshes/multicontact/downSlope2.s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

File: urdf/multicontact/downSlope_easy.urdf (robot description, URDF)
Before this commit: robot stair_bauzil, 1 links, 0 joints
Links:
- link base_link: geometry collision mesh filename=package://hpp_environments/meshes/multicontact/downSlope_ea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; visual mesh filename=package://hpp_environments/meshes/multicontact/downSlope_ea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

File: urdf/multicontact/downSlope_easy20.urdf (robot description, URDF)
Before this commit: robot stair_bauzil, 1 links, 0 joints
Links:
- link base_link: geometry collision mesh filename=package://hpp_environments/meshes/multicontact/downSlope_ea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; visual mesh filename=package://hpp_environments/meshes/multicontact/downSlope_ea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

File: urdf/multicontact/flat_hole.urdf (robot description, URDF)
Before this commit: robot flat_hole, 1 links, 0 joints
Links:
- link base_link: geometry collision mesh filename=package://hpp_environments/meshes/multicontact/flat_hole.stl; visual mesh filename=package://hpp_environments/meshes/multicontact/flat_hole.stl

File: urdf/multicontact/flat_step.urdf (robot description, URDF)
Before this commit: robot chair, 1 links, 0 joints
Links:
- link base_link: geometry collision mesh filename=package://hpp_environments/meshes/multicontact/flat_step.stl; visual mesh filename=package://hpp_environments/meshes/multicontact/flat_step.stl
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