Commit message: updated plinth path

File: urdf/multicontact/ori_plinth.urdf (robot description, URDF)
Before this commit: robot ori_plinth, 1 links, 0 joints
Links:
- link base_link: geometry collision mesh filename=package://hpp_environments/meshes/multicontact/ori_plinth.s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; visual mesh filename=package://hpp_environments/meshes/multicontact/ori_plinth.s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
