Commit message: use meshes from example-robot-data

File: urdf/tests/baxter_simple.urdf (robot description, URDF)
Before this commit: robot baxter, 57 links, 56 joints
Links:
- link head: geometry collision sphere radius=0.001; visual mesh filename=package://example-robot-data/robots/baxter_description/mesh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
- link left_lower_elbow: geometry collision cylinder length=0.10 radius=0.06; visual mesh filename=package://example-robot-data/robots/baxter_description/mesh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
- link left_lower_forearm: geometry collision cylinder length=0.10 radius=0.06; visual mesh filename=package://example-robot-data/robots/baxter_description/mesh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
- link left_lower_shoulder: geometry collision cylinder length=0.12 radius=0.06; visual mesh filename=package://example-robot-data/robots/baxter_description/mesh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
- link left_upper_elbow: geometry collision cylinder length=0.107 radius=0.06; visual mesh filename=package://example-robot-data/robots/baxter_description/mesh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
- link left_upper_forearm: geometry collision cylinder length=0.088 radius=0.06; visual mesh filename=package://example-robot-data/robots/baxter_description/mesh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
- link left_upper_shoulder: geometry collision cylinder length=0.2722 radius=0.06; visual mesh filename=package://example-robot-data/robots/baxter_description/mesh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
- link left_wrist: geometry collision cylinder length=0.165 radius=0.06; visual mesh filename=package://example-robot-data/robots/baxter_description/mesh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
- link pedestal: geometry collision mesh filename=package://example-robot-data/robots/baxter_description/mesh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; visual mesh filename=package://example-robot-data/robots/baxter_description/mesh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
- link right_lower_elbow: geometry collision cylinder length=0.10 radius=0.06; visual mesh filename=package://example-robot-data/robots/baxter_description/mesh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
- link right_lower_forearm: geometry collision cylinder length=0.10 radius=0.06; visual mesh filename=package://example-robot-data/robots/baxter_description/mesh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
- link right_lower_shoulder: geometry collision cylinder length=0.12 radius=0.06; visual mesh filename=package://example-robot-data/robots/baxter_description/mesh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
- link right_upper_elbow: geometry collision cylinder length=0.107 radius=0.06; visual mesh filename=package://example-robot-data/robots/baxter_description/mesh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
- link right_upper_forearm: geometry collision cylinder length=0.088 radius=0.06; visual mesh filename=package://example-robot-data/robots/baxter_description/mesh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
- link right_upper_shoulder: geometry collision cylinder length=0.2722 radius=0.06; visual mesh filename=package://example-robot-data/robots/baxter_description/mesh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
- link right_wrist: geometry collision cylinder length=0.165 radius=0.06; visual mesh filename=package://example-robot-data/robots/baxter_description/mesh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
- link screen: geometry collision sphere radius=0.001; visual mesh filename=package://example-robot-data/robots/baxter_description/mesh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
- link torso: geometry collision mesh filename=package://hpp_environments/meshes/tests/baxter_simple/torso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; visual mesh filename=package://example-robot-data/robots/baxter_description/mesh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
